Commit message: fix: car rear wheel isn't colliding with base

File: car.urdf (robot description, URDF)
Before this commit: robot romi, 4 links, 3 joints
Links:
- link wheel_rear: geometry collision cylinder length=0.01 radius=0.02; visual cylinder length=0.01 radius=0.02
Joints:
- joint wheel_rear_joint: origin xyz=0 -0.1 -0.024 rpy=0 1.57 0 -> xyz=0 -0.1 -0.03 rpy=0 1.57 0

Commit message: feat: attach load and increase friction on car

File: car.urdf (robot description, URDF)
Before this commit: robot romi, 4 links, 3 joints
Links:
- added link attached_load, mass 1.0; collision box size=0.1 0.15 0.05; visual box size=0.1 0.15 0.05
Joints:
- added joint attached_load_joint: type fixed, parent base_link, child attached_load, origin xyz=0 -0.05 0.025 rpy=0 0 0

Commit message: chore: rescale car to more accurate dims

File: car.urdf (robot description, URDF)
Before this commit: robot romi, 5 links, 4 joints
Links:
- link attached_load: geometry collision box size=0.05 0.075 0.025; visual box size=0.05 0.075 0.025
- link base_link: geometry collision cylinder length=0.01 radius=0.0825; visual cylinder length=0.01 radius=0.0825
- link wheel_l: geometry collision cylinder length=0.008 radius=0.035; visual cylinder length=0.008 radius=0.035
- link wheel_r: geometry collision cylinder length=0.008 radius=0.035; visual cylinder length=0.008 radius=0.035
- link wheel_rear: geometry collision cylinder length=0.01 radius=0.009; visual cylinder length=0.01 radius=0.009
Joints:
- joint attached_load_joint: origin xyz=0 -0.05 0.025 rpy=0 0 0 -> xyz=0 -0.025 0.0125 rpy=0 0 0
- joint wheel_l_joint: origin xyz=0.165 0 0 rpy=0 1.57 0 -> xyz=0.091 0 0.01 rpy=0 1.57 0
- joint wheel_r_joint: origin xyz=-0.165 0 0 rpy=0 1.57 0 -> xyz=-0.091 0 0.01 rpy=0 1.57 0
- joint wheel_rear_joint: origin xyz=0 -0.1 -0.03 rpy=0 1.57 0 -> xyz=0 -0.05 -0.0152 rpy=0 1.57 0
