Commit message: chore: upgrade gripper and increase errors for sim to real gap

File: python/urdf/car_gripper.urdf (robot description, URDF)
Before this commit: robot romi, 6 links, 5 joints
Links:
- link base_link: geometry collision mesh filename=base.stl; visual mesh filename=base.stl
Joints:
- joint gripper_joint: origin xyz=0 -0.0825 0.005 rpy=0 0 3.142 -> xyz=0 -0.085 0.005 rpy=0 0 3.142
- joint wheel_l_joint: origin xyz=0.091 0 0.01 rpy=0 1.57 0 -> xyz=0.0705 0 0.01 rpy=0 1.57 0
- joint wheel_r_joint: origin xyz=-0.091 0 0.01 rpy=0 1.57 0 -> xyz=-0.0705 0 0.01 rpy=0 1.57 0

Commit message: feat: train multi-object with closest point obs

File: python/urdf/car_gripper.urdf (robot description, URDF)
Before this commit: robot romi, 6 links, 5 joints
Links:
- added link gripper_centre_point, mass 0.1; collision sphere radius=0.005
Joints:
- added joint gripper_centre_point_joint: type fixed, parent base_link, child gripper_centre_point, origin xyz=0 -0.085 0.005 rpy=0 0 0

Commit message: Revert "feat: train multi-object with closest point obs"
This reverts commit f888294cc2baaadf25695900be4cff90e1d03d8c.

File: python/urdf/car_gripper.urdf (robot description, URDF)
Before this commit: robot romi, 7 links, 6 joints
Links:
- removed link gripper_centre_point
Joints:
- removed joint gripper_centre_point_joint
