Commit message: feat: train policy from images (not working)

File: python/rl_car/src/rl_car/urdf/car_gripper.urdf (robot description, URDF)
Before this commit: robot romi, 6 links, 5 joints
Links:
- link attached_load: geometry collision box size=0.075 0.05 0.025; visual box size=0.075 0.05 0.025
Joints:
- joint attached_load_joint: origin xyz=0 -0.025 0.0125 rpy=0 0 0 -> xyz=0 -0.015 0.0125 rpy=0 0 0
- joint gripper_joint: origin xyz=0 -0.085 0.005 rpy=0 0 3.142 -> xyz=0 -0.1 0.005 rpy=0 0 3.142

Commit message: feat: clear sim2real gap with image augmentation

File: python/rl_car/src/rl_car/urdf/car_gripper.urdf (robot description, URDF)
Before this commit: robot romi, 6 links, 5 joints
Links:
- link attached_load: geometry collision box size=0.08 0.06 0.025; visual box size=0.08 0.06 0.025

Commit message: chore: update robot urdf

File: python/rl_car/src/rl_car/urdf/car_gripper.urdf (robot description, URDF)
Before this commit: robot romi, 6 links, 5 joints
Links:
- added link roof_link, mass 0.1; collision mesh filename=roof.stl; visual mesh filename=roof.stl
Joints:
- added joint roof_joint: type fixed, parent base_link, child roof_link, origin xyz=0 0 0.045 rpy=0 0 0
